File: PCB/v2/Mouse_Emulator_V_2.sch (KiCad schematic (older format))
At the start: 31 parts, among them SW6 Rotary_Encoder_Switch, U1 STM32F103C8T6 (BluePill)

Commit message: Schematic
Parts:
- removed C1, C2, C3, C4, C5, C8, C9: 100nF, symbol Device:C
- removed C10: 10uF, symbol Device:CP
- removed D1: LED, symbol Device:LED
- removed DOWN: SW_Push_2, symbol Switch:SW_Push
- removed LEFT: SW_Push_3, symbol Switch:SW_Push
- removed MOUSE_CLICK: SW_Push_5, symbol Switch:SW_Push
- removed R1, R2, R3, R4, R5: 4K7, symbol Device:R
- removed R10, R12, R13, R15, R16, R6, R7, R8, R9: 10K, symbol Device:R
- removed R17: 470R, symbol Device:R
- removed RIGHT: SW_PUSH_4, symbol Switch:SW_Push
- removed U1: STM32F103C8T6 (BluePill), Package_QFP:LQFP-48_7x7mm_P0.5mm, symbol MCU_ST_STM32F1:STM32F103C8Tx
- removed UP: SW_Push_1, symbol Switch:SW_Push
- added C1, C2, C3, C4, C5, C6, C7, C8: 100n, symbol Device:C_Small
- added D1: RED, symbol Device:LED_Small
- added J1: JTAG, symbol Connector_Generic:Conn_01x04
- added R1: 1k5, symbol Device:R_Small
- added R10, R11, R12, R13, R2, R3, R4, R5, R6, R7, R8, R9: 10k, symbol Device:R_Small
- added R14: 4k7, symbol Device:R_Small
- added SW1: upSwitch, symbol Switch:SW_SPST
- added SW2: downSwitch, symbol Switch:SW_SPST
- added SW3: leftSwitch, symbol Switch:SW_SPST
- added SW4: rightSwitch, symbol Switch:SW_SPST
- added SW5: mouseSwitch, symbol Switch:SW_SPST
- added U1: BluePill_STM32F103C8T6, BluePill_breakouts:BluePill_STM32F103C, symbol bluepill_breakouts:BluePill_STM32F103C
Connections:
- net labels added: +3.3V, DOWN_Button, GND, JTAG_RX, JTAG_TX, LEFT_Button, MOUSE_Button, RIGHT_Button, UP_Button, enc_A, enc_B, enc_Switch, status_LED
- net labels removed: Earth, PA11, PA12, PA15, PA8, PB12, PB13, PB14, PB15
- wire segments 81 -> 79
- no-connect marks 28 -> 25
Other:
- note added: "Switches - 01x02 Conncetor\nRottary Encoder + LED - 01x05 Connector"
- note removed: "Enkoder"
- note removed: "Reference decoupling"
- note removed: "Sklopke"
- note removed: "uC"

Commit message: Schematic V2
Parts:
- removed C7, C8: 100n, symbol Device:C_Small
- removed D1: RED, symbol Device:LED_Small
- removed R13: 10k, symbol Device:R_Small
- removed R14: 4k7, symbol Device:R_Small
- removed SW1: upSwitch, symbol Switch:SW_SPST
- removed SW2: downSwitch, symbol Switch:SW_SPST
- removed SW3: leftSwitch, symbol Switch:SW_SPST
- removed SW4: rightSwitch, symbol Switch:SW_SPST
- removed SW5: mouseSwitch, symbol Switch:SW_SPST
- removed SW6: Rotary_Encoder_Switch, symbol Device:Rotary_Encoder_Switch
- added C? (x2): 100n, symbol Device:C_Small
- added J? (x5): Conn_01x02, symbol Connector_Generic:Conn_01x02
- added J?: Conn_01x06, symbol Connector_Generic:Conn_01x06
- added R?: 10k, symbol Device:R_Small
- added R?: 4k7, symbol Device:R_Small
Connections:
- net status_LED is gone; now on net LED_STATUS: U1.4 (PC15)
- net +3V3: now also J?.2 (Pin_2), J?.2 (Pin_2), J?.2 (Pin_2), J?.2 (Pin_2), J?.2 (Pin_2)
- net GND: now also C?.2, C?.2, J?.4 (Pin_4), J?.5 (Pin_5); no longer R1.1
- net at R2.1, R5.1: now also J?.1 (Pin_1)
- net ENC_A_CONN: now reaches R12.2
- net ENC_A_CONN: now also J?.1 (Pin_1)
- net at R3.1, R6.1: now also J?.1 (Pin_1)
- net at R4.1, R7.1: now also J?.1 (Pin_1)
- net at R10.1, R8.1: now also J?.1 (Pin_1)
- net at R11.1, R9.1: now also J?.1 (Pin_1)
- net LED_STATUS: now reaches R1.2
- net LED_STATUS: now also J?.6 (Pin_6)
- net DOWN_Button renamed DOWN_SWITCH
- net LEFT_Button renamed LEFT_SWITCH
- net MOUSE_Button renamed MOUSE_SWITCH
- net RIGHT_Button renamed RIGHT_SWITCH
- net UP_Button renamed UP_SWITCH
- net enc_A renamed ENC_A
- net enc_B renamed ENC_B
- net ENC_B: now also C?.1, R?.1
- net enc_Switch renamed ENC_SWITCH
- net ENC_SWITCH: now also C?.1, R?.1
- new net ENC_B_CONN: J?.2 (Pin_2), R?.2
- new net ENC_SWITCH_CONN: J?.3 (Pin_3), R?.2
- new net LED_STATUS_CONN: R1.1
Other:
- note added: "Connectors"
- note added: "Direction Switches"
- note added: "Microcontroller"
- note added: "Rottary Encoder + Status LED"
- note removed: "Switches - 01x02 Conncetor\nRottary Encoder + LED - 01x05 Connector"
- moved on the sheet: C1, C2, C3, C4, C5, C6, J1, R1, R10, R11, R12, R2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

Commit message: Pins definition + Schematic
Parts:
- added J8: Encoder_2, symbol Connector_Generic:Conn_01x04
- added SW1: Rotary_Encoder_Switch, symbol Device:Rotary_Encoder_Switch
- J1: renamed from J?; value Conn_01x02 -> UP_SWITCH
- J2: renamed from J?; value Conn_01x02 -> DOWN_SWITCH
- J3: renamed from J?; value Conn_01x02 -> LEFT_SWITCH
- J4: renamed from J?; value Conn_01x02 -> RIGHT_SWITCH
- J5: renamed from J?; value Conn_01x02 -> MOUSE_SWITCH
- J7: renamed from J?; value Conn_01x06 -> Encoder + LED
- U1: symbol bluepill_breakouts:BluePill_STM32F103C -> Mouse_Emulator_V_2-rescue:BluePill_STM32F103C-bluepill_breakouts
- gave numbers to parts that had none: 4
- renumbered J1 to J6, R2 to R1, R11 to R10, R1 to R11, R3 to R2, R4 to R3, R5 to R4, R6 to R5, R7 to R6, R8 to R7, R9 to R8, R10 to R9
Connections:
- net +3V3: now also U1.40 (VCC3V3); no longer U1.39 (GND)
- net GND: now also U1.39 (GND), J8.4 (Pin_4), SW1.C, SW1.S2; no longer U1.40 (VCC3V3)
- net JTAG_RX: now also J6.2 (Pin_2), U1.26 (PA9_RX1); no longer J6.3 (Pin_3), U1.27 (PA10_RX1)
- net JTAG_TX: now also J6.3 (Pin_3), U1.27 (PA10_TX1); no longer J6.2 (Pin_2), U1.26 (PA9_TX1)
- net LEFT_SWITCH: now also U1.16 (PB11_SDA2); no longer U1.23 (PB14_MISO2)
- net MOUSE_SWITCH: now also U1.23 (PB14_MISO2); no longer U1.25 (PA8)
- net RIGHT_SWITCH: now also U1.15 (PB10_SCL2); no longer U1.24 (PB15_MOSI2)
- new net ENC_A_CONN2: J8.1 (Pin_1), SW1.A
- new net ENC_B_CONN2: J8.2 (Pin_2), SW1.B
- new net ENC_SWITCH_CONN2: J8.3 (Pin_3), SW1.S1
Other:
- note added: "Rottary Encoder (Small PCB)"
- moved on the sheet: C6, C7, C8, J6, J7, R11, R12, R13, R14
